Commit message: change to new urdf

File: maniptrans_envs/assets/wujihand/urdf/left.urdf (robot description, URDF)
Before this commit: robot wujihand-left-v1.0.0, 26 links, 25 joints
Links:
- link finger1_link1: geometry collision mesh filename=mesh_soft_body/left/left_finger1_link1.stl; visual mesh filename=mesh_soft_body/left/left_finger1_link1.stl
- link finger1_link2: geometry collision mesh filename=mesh_soft_body/left/left_finger1_link2.stl; visual mesh filename=mesh_soft_body/left/left_finger1_link2.stl
- link finger1_link3: geometry collision mesh filename=mesh_soft_body/left/left_finger1_link3.stl; visual mesh filename=mesh_soft_body/left/left_finger1_link3.stl
- link finger1_link4: geometry collision mesh filename=mesh_soft_body/left/left_finger1_link4.stl; visual mesh filename=mesh_soft_body/left/left_finger1_link4.stl
- link finger1_tip_link: mass 0.004 -> 0.0041; geometry 
- link finger2_link1: geometry collision mesh filename=mesh_soft_body/left/left_finger2_link1.stl; visual mesh filename=mesh_soft_body/left/left_finger2_link1.stl
- link finger2_link2: geometry collision mesh filename=mesh_soft_body/left/left_finger2_link2.stl; visual mesh filename=mesh_soft_body/left/left_finger2_link2.stl
- link finger2_link3: geometry collision mesh filename=mesh_soft_body/left/left_finger2_link3.stl; visual mesh filename=mesh_soft_body/left/left_finger2_link3.stl
- link finger2_link4: geometry collision mesh filename=mesh_soft_body/left/left_finger2_link4.stl; visual mesh filename=mesh_soft_body/left/left_finger2_link4.stl
- link finger2_tip_link: mass 0.004 -> 0.00318; geometry 
- link finger3_link1: geometry collision mesh filename=mesh_soft_body/left/left_finger3_link1.stl; visual mesh filename=mesh_soft_body/left/left_finger3_link1.stl
- link finger3_link2: geometry collision mesh filename=mesh_soft_body/left/left_finger3_link2.stl; visual mesh filename=mesh_soft_body/left/left_finger3_link2.stl
- link finger3_link3: geometry collision mesh filename=mesh_soft_body/left/left_finger3_link3.stl; visual mesh filename=mesh_soft_body/left/left_finger3_link3.stl
- link finger3_link4: geometry collision mesh filename=mesh_soft_body/left/left_finger3_link4.stl; visual mesh filename=mesh_soft_body/left/left_finger3_link4.stl
- link finger3_tip_link: mass 0.004 -> 0.00318; geometry 
- link finger4_link1: geometry collision mesh filename=mesh_soft_body/left/left_finger4_link1.stl; visual mesh filename=mesh_soft_body/left/left_finger4_link1.stl
- link finger4_link2: geometry collision mesh filename=mesh_soft_body/left/left_finger4_link2.stl; visual mesh filename=mesh_soft_body/left/left_finger4_link2.stl
- link finger4_link3: geometry collision mesh filename=mesh_soft_body/left/left_finger4_link3.stl; visual mesh filename=mesh_soft_body/left/left_finger4_link3.stl
- link finger4_link4: geometry collision mesh filename=mesh_soft_body/left/left_finger4_link4.stl; visual mesh filename=mesh_soft_body/left/left_finger4_link4.stl
- link finger4_tip_link: mass 0.004 -> 0.00318; geometry 
- link finger5_link1: geometry collision mesh filename=mesh_soft_body/left/left_finger5_link1.stl; visual mesh filename=mesh_soft_body/left/left_finger5_link1.stl
- link finger5_link2: geometry collision mesh filename=mesh_soft_body/left/left_finger5_link2.stl; visual mesh filename=mesh_soft_body/left/left_finger5_link2.stl
- link finger5_link3: geometry collision mesh filename=mesh_soft_body/left/left_finger5_link3.stl; visual mesh filename=mesh_soft_body/left/left_finger5_link3.stl
- link finger5_link4: geometry collision mesh filename=mesh_soft_body/left/left_finger5_link4.stl; visual mesh filename=mesh_soft_body/left/left_finger5_link4.stl
- link finger5_tip_link: mass 0.004 -> 0.00318; geometry 
- link palm_link: mass 0.2179 -> 0.16914; geometry collision mesh filename=mesh_soft_body/left/left_palm_link.stl; visual mesh filename=mesh_soft_body/left/left_palm_link.stl
Joints:
- joint finger1_joint1: axis -0 1 -0 -> 0 -1 0; limit lower=-0.0448 upper=1.6508 effort=0.6 velocity=8.58701992 -> lower=0.0475 upper=1.6033 effort=0.4452 velocity=8.587; origin xyz=0.0085244 -0.020575 0.028712 rpy=1.328 -0.37161 0.7307 -> xyz=0.00843985365415843 -0.0205866432296062 0.0288928344146015 rpy=-1.32802443797267 0.371613529401196 -2.41089218263562
- joint finger1_joint2: axis -1 0 0 -> 0 0.999999999999998 0; limit lower=-0.1659 upper=0.9339 effort=0.6 velocity=11.10029404 -> lower=-0.1387 upper=0.9324 effort=0.4259 velocity=11.1; origin xyz=-0.0047549 0.0060191 0.014132 rpy=-0.27968 -0.55633 -0.081982 -> xyz=0.00475489639781444 -0.00581913884095369 0.0141320959775981 rpy=-0.574275017658819 0.236773443835485 -1.80339762361133
- joint finger1_joint3: limit lower=-0.4932 upper=1.6272 effort=0.3 velocity=12.86307659 -> lower=-0.4642 upper=1.5623 effort=0.1888 velocity=12.863; origin xyz=0.0009915 -0.00026671 0.033166 rpy=-0.049049 0.017311 0.33774 -> xyz=-0.000266710475105365 -0.000991501671842022 0.0346656206595102 rpy=-0.0490495013721327 0.0173112654625817 -1.23305223942119
- joint finger1_joint4: limit lower=-0.4932 upper=1.6272 effort=0.3 velocity=13.57866158 -> lower=-0.4699 upper=1.5568 effort=0.1468 velocity=13.578; origin xyz=0 4.0225E-05 0.028987 rpy=0 0 0 -> xyz=0 -0.000200000007014417 0.0294999998969491 rpy=0 0 0
- joint finger1_tip_fixed: limit lower=-0.5236 upper=0.5236 effort=100 velocity=10 -> (none); origin xyz=-0.001058 -0.00044022 0.029313 rpy=0 0 0 -> xyz=-0.00104999999999688 0.000200000000001237 0.0272999999999996 rpy=0 0 0
- joint finger2_joint1: limit lower=-0.32695 upper=1.63595 effort=1 velocity=8.203047484 -> lower=-0.1585 upper=1.5604 effort=0.6188 velocity=8.203; origin xyz=-0.0058701 -0.029434 0.091917 rpy=0.11071 -0.071133 0.21823 -> xyz=-0.00587008921405553 -0.0294338632807666 0.0919165306703556 rpy=0.110709291859976 -0.0711392444947576 0.218224846837306
- joint finger2_joint2: axis -1 -0 -0 -> 0 1 0; limit lower=-0.495 upper=0.495 effort=0.2 velocity=8.115781022 -> lower=-0.37 upper=0.37 effort=0.1822 velocity=8.115; origin xyz=0.0022 0 0.004 rpy=-0.00043322 1.0969E-05 0 -> xyz=0.00220000016133353 0 0.00400000572577126 rpy=0 0 1.57079631622159
- joint finger2_joint3: axis -0 1 -0 -> 0 1 0; limit lower=-0.4932 upper=1.6272 effort=0.3 velocity=12.86307659 -> lower=-0.4777 upper=1.5485 effort=0.2251 velocity=12.863; origin xyz=-0.0046 0 0.036618 rpy=0 0 -0.00026861 -> xyz=0 0.00474999948522651 0.0436176874464638 rpy=0 0 -1.57052771407713
- joint finger2_joint4: axis -0 1 -0 -> 0 1 0; limit lower=-0.4932 upper=1.6272 effort=0.3 velocity=13.57866158 -> lower=-0.4683 upper=1.5753 effort=0.2170 velocity=13.578; origin xyz=0 0 0.029 rpy=0 0 0 -> xyz=0 -0.00020000000114569 0.0295000000005511 rpy=0 0 0
- joint finger2_tip_fixed: origin xyz=-0.0010404 0 0.0267 rpy=0 0 0 -> xyz=-0.00105210040162161 0.000210869249702341 0.0266999998503596 rpy=0 0 0
- joint finger3_joint1: axis -0 1 -0 -> 0 1 0; limit lower=-0.32695 upper=1.63595 effort=1 velocity=8.203047484 -> lower=-0.1644 upper=1.5516 effort=0.6494 velocity=8.203; origin xyz=-0.01046 -0.0074615 0.089544 rpy=5.0886E-05 -0.087266 -0.00058387 -> xyz=-0.0104597238646911 -0.00746146014383039 0.0895435117684639 rpy=5.08943582386716E-05 -0.0872664620461616 -0.000583871753342456
- joint finger3_joint2: axis -1 0 0 -> 0 1 0; limit lower=-0.495 upper=0.495 effort=0.2 velocity=8.115781022 -> lower=-0.37 upper=0.37 effort=0.1827 velocity=8.115; origin xyz=0.0022 0 0.004 rpy=-0.00043323 0 0 -> xyz=0.00220000043882706 0 0.0040000056099367 rpy=0 0 1.57079631623283
- joint finger3_joint3: axis -0 1 -0 -> 0 1 0; limit lower=-0.4932 upper=1.6272 effort=0.3 velocity=12.86307659 -> lower=-0.4739 upper=1.5512 effort=0.2078 velocity=12.863; origin xyz=-0.0046 0 0.036618 rpy=0 0 -0.00026862 -> xyz=0 0.00474999936719482 0.0436176874471427 rpy=0 0 -1.57052771407715
- joint finger3_joint4: axis -0 1 -0 -> 0 1 0; limit lower=-0.4932 upper=1.6272 effort=0.3 velocity=13.57866158 -> lower=-0.4684 upper=1.5745 effort=0.2018 velocity=13.578; origin xyz=0 0 0.029 rpy=0 0 0 -> xyz=0 -0.000200000001145385 0.029499999999373 rpy=0 0 0
- joint finger3_tip_fixed: origin xyz=-0.0010404 0 0.0267 rpy=0 0 0 -> xyz=-0.00105039969315103 0.000202672284305974 0.0266999998510997 rpy=0 0 0
- joint finger4_joint1: axis -0 1 -0 -> 0 1 0; limit lower=-0.32695 upper=1.63595 effort=1 velocity=8.203047484 -> lower=-0.1554 upper=1.5585 effort=0.6389 velocity=8.203; origin xyz=-0.0076649 0.013712 0.084429 rpy=-0.090379 -0.084038 -0.047072 -> xyz=-0.00766485992731566 0.0137122383759935 0.0844286945869771 rpy=-0.0903746132831303 -0.0834355016926537 -0.0471266291492555
- joint finger4_joint2: axis -1 0 0 -> 0 1 0; limit lower=-0.495 upper=0.495 effort=0.2 velocity=8.115781022 -> lower=-0.37 upper=0.37 effort=0.1832 velocity=8.115; origin xyz=0.0022024 0 0.0039987 rpy=-0.00043323 0.00060486 0 -> xyz=0.00220000046883515 0 0.00400000548163587 rpy=0 0 1.57079631622036
- joint finger4_joint3: axis -0 1 -0 -> 0 1 0; limit lower=-0.4932 upper=1.6272 effort=0.3 velocity=12.86307659 -> lower=-0.4765 upper=1.5487 effort=0.2249 velocity=12.863; origin xyz=-0.0046 0 0.036618 rpy=0 0 -0.00026862 -> xyz=0 0.00474999947605386 0.0436176874464634 rpy=0 0 -1.5705277035072
- joint finger4_joint4: axis -0 1 -0 -> 0 1 0; limit lower=-0.4932 upper=1.6272 effort=0.3 velocity=13.57866158 -> lower=-0.4777 upper=1.5634 effort=0.2044 velocity=13.578; origin xyz=0 0 0.029 rpy=0 0 0 -> xyz=0 -0.000200000001146229 0.0294999999999928 rpy=0 0 0
- joint finger4_tip_fixed: origin xyz=-0.0010993 0 0.026698 rpy=0 0 0 -> xyz=-0.00104998290825126 0.000202557162358057 0.0266999998509249 rpy=0 0 0
- joint finger5_joint1: limit lower=-0.32695 upper=1.63595 effort=1 velocity=8.203047484 -> lower=-0.1626 upper=1.5585 effort=0.6441 velocity=8.203; origin xyz=-0.0022687 0.034001 0.074281 rpy=-0.1925 -0.09326 -0.15753 -> xyz=-0.00226865105942822 0.0340011106647859 0.0742813381432916 rpy=-0.192483650752976 -0.0925172324525506 -0.157672818923778
- joint finger5_joint2: axis -1 0 0 -> 0 1 0; limit lower=-0.495 upper=0.495 effort=0.2 velocity=8.115781022 -> lower=-0.37 upper=0.37 effort=0.1798 velocity=8.115; origin xyz=0.002203 0 0.0039983 rpy=-0.00043323 0.00075655 0 -> xyz=0.0022000006386125 0 0.0040000052815589 rpy=0 0 1.57079631621958
- joint finger5_joint3: axis -0 1 -0 -> 0 1 0; limit lower=-0.4932 upper=1.6272 effort=0.3 velocity=12.86307659 -> lower=-0.4768 upper=1.5490 effort=0.2384 velocity=12.863; origin xyz=-0.0046 0 0.036618 rpy=0 0 -0.00026862 -> xyz=0 0.00474999955614431 0.0436176864501152 rpy=0 0 -1.57052771407715
- joint finger5_joint4: axis -0 1 -0 -> 0 1 0; limit lower=-0.4932 upper=1.6272 effort=0.3 velocity=13.57866158 -> lower=-0.4683 upper=1.5735 effort=0.1866 velocity=13.578; origin xyz=0 0 0.029 rpy=0 0 0 -> xyz=0 -0.000200000001688738 0.0295000009963858 rpy=0 0 0
- joint finger5_tip_fixed: limit effort=100 velocity=10 -> (none); origin xyz=-0.0011127 0 0.026697 rpy=0 0 0 -> xyz=-0.00105040660537688 0.000201047212892366 0.0266999998509271 rpy=0 0 0

File: maniptrans_envs/assets/wujihand/urdf/right.urdf (robot description, URDF)
Before this commit: robot wujihand-right-v1.0.0, 26 links, 25 joints
Links:
- link finger1_link1: geometry collision mesh filename=mesh_soft_body/right/finger1_link1.stl; visual mesh filename=mesh_soft_body/right/finger1_link1.stl
- link finger1_link2: geometry collision mesh filename=mesh_soft_body/right/finger1_link2.stl; visual mesh filename=mesh_soft_body/right/finger1_link2.stl
- link finger1_link3: geometry collision mesh filename=mesh_soft_body/right/finger1_link3.stl; visual mesh filename=mesh_soft_body/right/finger1_link3.stl
- link finger1_link4: geometry collision mesh filename=mesh_soft_body/right/finger1_link4.stl; visual mesh filename=mesh_soft_body/right/finger1_link4.stl
- link finger1_tip_link: mass 0.004 -> 0.0041; geometry 
- link finger2_link1: geometry collision mesh filename=mesh_soft_body/right/finger2_link1.stl; visual mesh filename=mesh_soft_body/right/finger2_link1.stl
- link finger2_link2: geometry collision mesh filename=mesh_soft_body/right/finger2_link2.stl; visual mesh filename=mesh_soft_body/right/finger2_link2.stl
- link finger2_link3: geometry collision mesh filename=mesh_soft_body/right/finger2_link3.stl; visual mesh filename=mesh_soft_body/right/finger2_link3.stl
- link finger2_link4: geometry collision mesh filename=mesh_soft_body/right/finger2_link4.stl; visual mesh filename=mesh_soft_body/right/finger2_link4.stl
- link finger2_tip_link: mass 0.004 -> 0.00318; geometry 
- link finger3_link1: geometry collision mesh filename=mesh_soft_body/right/finger3_link1.stl; visual mesh filename=mesh_soft_body/right/finger3_link1.stl
- link finger3_link2: geometry collision mesh filename=mesh_soft_body/right/finger3_link2.stl; visual mesh filename=mesh_soft_body/right/finger3_link2.stl
- link finger3_link3: geometry collision mesh filename=mesh_soft_body/right/finger3_link3.stl; visual mesh filename=mesh_soft_body/right/finger3_link3.stl
- link finger3_link4: geometry collision mesh filename=mesh_soft_body/right/finger3_link4.stl; visual mesh filename=mesh_soft_body/right/finger3_link4.stl
- link finger3_tip_link: mass 0.004 -> 0.00318; geometry 
- link finger4_link1: geometry collision mesh filename=mesh_soft_body/right/finger4_link1.stl; visual mesh filename=mesh_soft_body/right/finger4_link1.stl
- link finger4_link2: geometry collision mesh filename=mesh_soft_body/right/finger4_link2.stl; visual mesh filename=mesh_soft_body/right/finger4_link2.stl
- link finger4_link3: geometry collision mesh filename=mesh_soft_body/right/finger4_link3.stl; visual mesh filename=mesh_soft_body/right/finger4_link3.stl
- link finger4_link4: geometry collision mesh filename=mesh_soft_body/right/finger4_link4.stl; visual mesh filename=mesh_soft_body/right/finger4_link4.stl
- link finger4_tip_link: mass 0.004 -> 0.00318; geometry 
- link finger5_link1: geometry collision mesh filename=mesh_soft_body/right/finger5_link1.stl; visual mesh filename=mesh_soft_body/right/finger5_link1.stl
- link finger5_link2: geometry collision mesh filename=mesh_soft_body/right/finger5_link2.stl; visual mesh filename=mesh_soft_body/right/finger5_link2.stl
- link finger5_link3: geometry collision mesh filename=mesh_soft_body/right/finger5_link3.stl; visual mesh filename=mesh_soft_body/right/finger5_link3.stl
- link finger5_link4: geometry collision mesh filename=mesh_soft_body/right/finger5_link4.stl; visual mesh filename=mesh_soft_body/right/finger5_link4.stl
- link finger5_tip_link: mass 0.004 -> 0.00318; geometry 
- link palm_link: mass 0.2179 -> 0.16914; geometry collision mesh filename=mesh_soft_body/right/palm_link.stl; visual mesh filename=mesh_soft_body/right/palm_link.stl
Joints:
- joint finger1_joint1: limit lower=-0.0448 upper=1.6508 effort=0.6 velocity=8.58701992 -> lower=0.0368 upper=1.6125 effort=0.4452 velocity=8.58701992; origin xyz=0.00852444051536966 0.0205754004992104 0.0287119465316217 rpy=-1.32802443797267 -0.371613529401197 -0.730700470955738 -> xyz=0.0085244 0.020575 0.028712 rpy=-1.328 -0.37161 -0.7307
- joint finger1_joint2: limit lower=-0.1659 upper=0.9339 effort=0.6 velocity=11.10029404 -> lower=-0.1576 upper=0.9312 effort=0.4259 velocity=11.10029404; origin xyz=-0.00475489770145063 -0.00601914141399163 0.0141320977109324 rpy=-0.574275025049342 -0.236773483165492 1.80339766411149 -> xyz=-0.0047549 -0.0060191 0.014132 rpy=-0.57428 -0.23677 1.8034
- joint finger1_joint3: limit lower=-0.4932 upper=1.6272 effort=0.3 velocity=12.86307659 -> lower=-0.4638 upper=1.5607 effort=0.1888 velocity=12.86307659; origin xyz=0.00026670985188593 -0.000991501581071832 0.0331656190850421 rpy=0.0490494507279603 0.0173112436656061 -1.90854042682209 -> xyz=0.00018873 -0.0009916 0.034664 rpy=0.049049 0.017311 -1.9085
- joint finger1_joint4: limit lower=-0.4932 upper=1.6272 effort=0.3 velocity=13.57866158 -> lower=-0.4829 upper=1.5451 effort=0.1468 velocity=13.57866158; origin xyz=0 -5.00007422951686E-05 0.0289999996622586 rpy=0 0 0 -> xyz=0 -0.00025 0.0295 rpy=0 0 0
- joint finger1_tip_fixed: limit lower=0 upper=0 effort=100 velocity=10 -> (none); origin xyz=-0.00104623528319934 0.000443681117589321 0.0293000000558906 rpy=0 0 0 -> xyz=-0.0011048 0.00023218 0.0283 rpy=0 0 0
- joint finger2_joint1: axis 0 0.999999906158207 0.000433224625971368 -> 0 1 0; limit lower=-0.32695 upper=1.63595 effort=1 velocity=8.203047484 -> lower=-0.1611 upper=1.5588 effort=0.6188 velocity=8.203047484; origin xyz=-0.00587008921485247 0.0294338632809287 0.0919165306699325 rpy=-0.111142508461784 -0.0711392477320386 -0.218224846477167 -> xyz=-0.0058701 0.029434 0.091917 rpy=-0.11071 -0.071139 -0.21822
- joint finger2_joint2: axis -0.999999999978991 0 0 -> -1 0 0; limit lower=-0.495 upper=0.495 effort=0.2 velocity=8.115781022 -> lower=-0.4044 upper=0.3054 effort=0.1822 velocity=8.115781022; origin xyz=0.00220000017524629 0 0.00400000534382478 rpy=0.000433224548403847 0 0 -> xyz=0.0022 0 0.004 rpy=0 0 0
- joint finger2_joint3: limit lower=-0.4932 upper=1.6272 effort=0.3 velocity=12.86307659 -> lower=-0.4714 upper=1.5504 effort=0.2251 velocity=12.86307659; origin xyz=-0.00460023735005808 1.55817705260984E-05 0.0366176526568538 rpy=-0.000433222790942502 0 -0.000268612691124751 -> xyz=-0.0047503 0 0.043618 rpy=0 0 -0.00026861
- joint finger2_joint4: limit lower=-0.4932 upper=1.6272 effort=0.3 velocity=13.57866158 -> lower=-0.4644 upper=1.5753 effort=0.2170 velocity=13.57866158; origin xyz=0 0 0.0290000000150095 rpy=0 0 0 -> xyz=0 0 0.0295 rpy=0 0 0
- joint finger2_tip_fixed: limit lower=0 upper=0 effort=100 velocity=10 -> (none); origin xyz=-0.00104999539509563 0 0.0274000004481596 rpy=0 0 0 -> xyz=-0.00105 0 0.0274 rpy=0 0 0
- joint finger3_joint1: axis 0 0.999999906158095 0.000433224884501103 -> 0 1 0; limit lower=-0.32695 upper=1.63595 effort=1 velocity=8.203047484 -> lower=-0.1719 upper=1.5496 effort=0.6494 velocity=8.203047484; origin xyz=-0.0104597238611628 0.00746146014385576 0.0895435117703666 rpy=-0.00048411119168703 -0.087266465303481 0.000583871740106801 -> xyz=-0.01046 0.0074615 0.089544 rpy=-5.0886E-05 -0.087266 0.00058387
- joint finger3_joint2: limit lower=-0.495 upper=0.495 effort=0.2 velocity=8.115781022 -> lower=-0.4014 upper=0.2996 effort=0.1827 velocity=8.115781022; origin xyz=0.0022000005026625 0 0.00400000522628907 rpy=0.000433224806924388 0 0 -> xyz=0.0022 0 0.004 rpy=0 0 0
- joint finger3_joint3: limit lower=-0.4932 upper=1.6272 effort=0.3 velocity=12.86307659 -> lower=-0.4632 upper=1.5613 effort=0.2078 velocity=12.86307659; origin xyz=-0.00460000064410125 1.55817799863825E-05 0.036617682393194 rpy=-0.000433224785853114 0 -0.000268612686864552 -> xyz=-0.00475 0 0.043618 rpy=0 0 -0.00026861
- joint finger3_joint4: limit lower=-0.4932 upper=1.6272 effort=0.3 velocity=13.57866158 -> lower=-0.4697 upper=1.5702 effort=0.2018 velocity=13.57866158; origin xyz=0 0 0.0290000000150094 rpy=0 0 0 -> xyz=0 0 0.0295 rpy=0 0 0
- joint finger3_tip_fixed: limit lower=0 upper=0 effort=100 velocity=10 -> (none); origin xyz=-0.00104042865141054 0 0.0267000008801756 rpy=0 0 0 -> xyz=-0.0010491 0 0.0267 rpy=0 0 0
- joint finger4_joint1: axis 0 0.999999906157892 0.000433225355001288 -> -0 1 -0; limit lower=-0.32695 upper=1.63595 effort=1 velocity=8.203047484 -> lower=-0.1601 upper=1.5534 effort=0.6389 velocity=8.203047484; origin xyz=-0.0076648599285041 -0.0137122383759844 0.084428694586379 rpy=0.0899413960034348 -0.0834355049367681 0.0471266288536016 -> xyz=-0.0076649 -0.013712 0.084429 rpy=0.090375 -0.083436 0.047127
- joint finger4_joint2: limit lower=-0.495 upper=0.495 effort=0.2 velocity=8.115781022 -> lower=-0.4134 upper=0.3161 effort=0.1832 velocity=8.115781022; origin xyz=0.00220000053755089 0 0.00400000510026774 rpy=0.000433225366118357 0 0 -> xyz=0.0022 0 0.004 rpy=0 0 0
- joint finger4_joint3: limit lower=-0.4932 upper=1.6272 effort=0.3 velocity=12.86307659 -> lower=-0.4782 upper=1.5448 effort=0.2249 velocity=12.86307659; origin xyz=-0.00459999999033558 1.55818004638833E-05 0.0366176824753135 rpy=-0.000433225349833524 0 -0.000268612687102299 -> xyz=-0.00475 0 0.043618 rpy=0 0 -0.00026861
- joint finger4_joint4: limit lower=-0.4932 upper=1.6272 effort=0.3 velocity=13.57866158 -> lower=-0.4825 upper=1.5550 effort=0.2044 velocity=13.57866158; origin xyz=0 0 0.0290000000150089 rpy=0 0 0 -> xyz=0 0 0.0295 rpy=0 0 0
- joint finger4_tip_fixed: limit lower=0 upper=0 effort=100 velocity=10 -> (none); origin xyz=-0.00104042861977702 0 0.026700000917914 rpy=0 0 0 -> xyz=-0.0010528 0 0.0267 rpy=0 0 0
- joint finger5_joint1: axis 0 0.999999906157892 0.000433225353070638 -> 0 1 0; limit lower=-0.32695 upper=1.63595 effort=1 velocity=8.203047484 -> lower=-0.1674 upper=1.5539 effort=0.6441 velocity=8.203047484; origin xyz=-0.00226865106062467 -0.0340011106648613 0.0742813381426987 rpy=0.192050433506504 -0.0925172356498861 0.157672818297325 -> xyz=-0.0022687 -0.034001 0.074281 rpy=0.19248 -0.092517 0.15767
- joint finger5_joint2: limit lower=-0.495 upper=0.495 effort=0.2 velocity=8.115781022 -> lower=-0.4203 upper=0.2931 effort=0.1798 velocity=8.115781022; origin xyz=0.00220000070730803 0 0.00400000490038611 rpy=0.000433225364229257 0 0 -> xyz=0.0022 0 0.004 rpy=0 0 0
- joint finger5_joint3: limit lower=-0.4932 upper=1.6272 effort=0.3 velocity=12.86307659 -> lower=-0.4804 upper=1.5420 effort=0.2384 velocity=12.86307659; origin xyz=-0.0046 1.5582E-05 0.036618 rpy=-0.00043323 0 -0.00026861 -> xyz=-0.00475 0 0.043618 rpy=0 0 -0.00026861
- joint finger5_joint4: limit lower=-0.4932 upper=1.6272 effort=0.3 velocity=13.57866158 -> lower=-0.4705 upper=1.5709 effort=0.1866 velocity=13.57866158; origin xyz=0 0 0.029 rpy=0 0 0 -> xyz=0 0 0.0295 rpy=0 0 0
- joint finger5_tip_fixed: limit lower=0 upper=0 effort=100 velocity=10 -> (none); origin xyz=-0.00104042861181322 0 0.0267000011472218 rpy=0 0 0 -> xyz=-0.0010446 1.1308E-05 0.0267 rpy=0 0 0
